File: kicad/rpipicow.kicad_sch (KiCad schematic)
At the start: 1 part, among them U4 RPi Pico W

Commit message: Updated board, using THT resistors, fixed wiring
Connections:
- net GND: now also U4.13 (GND3), U4.18 (GND4), U4.23 (GND5), U4.28 (GND6), U4.33 (GND7), U4.42 (GND_DEBUG), U4.8 (GND2)
Changed lines of the file:
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@@
   (title_block
     (title "mqtt-power-control-interface")
-    (date "2023-08-06")
-    (rev "1.0.0")
+    (date "2023-08-28")
+    (rev "1.1.0")
+  )
+  (wire (pts (xy 68.58 58.42) (xy 88.9 58.42))
+    (stroke (width 0) (type default))
   )
   (wire (pts (xy 74.93 73.66) (xy 68.58 73.66))
     (stroke (width 0) (type default))
   )
+  (wire (pts (xy 68.58 71.12) (xy 88.9 71.12))
+    (stroke (width 0) (type default))
+  )
+  (wire (pts (xy 22.86 58.42) (xy 43.18 58.42))
+    (stroke (width 0) (type default))
+  )
   (wire (pts (xy 74.93 63.5) (xy 68.58 63.5))
     (stroke (width 0) (type default))
@@
     (stroke (width 0) (type default))
   )
+  (wire (pts (xy 55.88 81.28) (xy 55.88 85.09))
+    (stroke (width 0) (type default))
+  )
+  (wire (pts (xy 68.58 45.72) (xy 88.9 45.72))
+    (stroke (width 0) (type default))
+  )
   (wire (pts (xy 36.83 68.58) (xy 43.18 68.58))
     (stroke (width 0) (type default))
@@
     (stroke (width 0) (type default))
   )
+  (wire (pts (xy 22.86 71.12) (xy 43.18 71.12))
+    (stroke (width 0) (type default))
+  )
   (wire (pts (xy 36.83 53.34) (xy 43.18 53.34))
     (stroke (width 0) (type default))
@@
     (stroke (width 0) (type default))
   )
+  (wire (pts (xy 22.86 45.72) (xy 43.18 45.72))
+    (stroke (width 0) (type default))
+  )
   (wire (pts (xy 36.83 55.88) (xy 43.18 55.88))
     (stroke (width 0) (type default))
@@
     (property "Intersheetrefs" "${INTERSHEET_REFS}" (at 26.9505 68.58 0)
       (effects (font (size 1.27 1.27)) (justify right) hide)
+    )
+  )
+  (symbol (lib_id "power:GND") (at 88.9 45.72 0) (unit 1)
+    (in_bom yes) (on_board yes) (dnp no) (fields_autoplaced)
+    (property "Reference" "#PWR013" (at 88.9 52.07 0)
+      (effects (font (size 1.27 1.27)) hide)
+    )
+    (property "Value" "GND" (at 88.9 50.8 0)
+      (effects (font (size 1.27 1.27)))
+    )
+    (property "Footprint" "" (at 88.9 45.72 0)
+      (effects (font (size 1.27 1.27)) hide)
+    )
+    (property "Datasheet" "" (at 88.9 45.72 0)
+      (effects (font (size 1.27 1.27)) hide)
+    )
+    (pin "1")
+    (instances
+      (project "mqtt-power-control-interface"
+        (path "/23700ef1-6085-46e5-b227-871d4be6e7a6"
+          (reference "#PWR013") (unit 1)
+        )
+        (path "/23700ef1-6085-46e5-b227-871d4be6e7a6/9a6b2a70-b072-4ffe-942c-277ad77cced3"
+          (reference "#PWR02") (unit 1)
+        )
+      )
+    )
+  )
+  (symbol (lib_id "power:GND") (at 22.86 58.42 0) (unit 1)
+    (in_bom yes) (on_board yes) (dnp no) (fields_autoplaced)
+    (property "Reference" "#PWR013" (at 22.86 64.77 0)
+      (effects (font (size 1.27 1.27)) hide)
+    )
+    (property "Value" "GND" (at 22.86 63.5 0)
+      (effects (font (size 1.27 1.27)))
+    )
+    (property "Footprint" "" (at 22.86 58.42 0)
+      (effects (font (size 1.27 1.27)) hide)
+    )
+    (property "Datasheet" "" (at 22.86 58.42 0)
+      (effects (font (size 1.27 1.27)) hide)
+    )
+    (pin "1")
+    (instances
+      (project "mqtt-power-control-interface"
+        (path "/23700ef1-6085-46e5-b227-871d4be6e7a6"
+          (reference "#PWR013") (unit 1)
+        )
+        (path "/23700ef1-6085-46e5-b227-871d4be6e7a6/9a6b2a70-b072-4ffe-942c-277ad77cced3"
+          (reference "#PWR06") (unit 1)
+        )
+      )
     )
   )
@@
     )
   )
+  (symbol (lib_id "power:GND") (at 88.9 58.42 0) (unit 1)
+    (in_bom yes) (on_board yes) (dnp no) (fields_autoplaced)
+    (property "Reference" "#PWR013" (at 88.9 64.77 0)
+      (effects (font (size 1.27 1.27)) hide)
+    )
+    (property "Value" "GND" (at 88.9 63.5 0)
+      (effects (font (size 1.27 1.27)))
+    )
+    (property "Footprint" "" (at 88.9 58.42 0)
+      (effects (font (size 1.27 1.27)) hide)
+    )
+    (property "Datasheet" "" (at 88.9 58.42 0)
+      (effects (font (size 1.27 1.27)) hide)
+    )
+    (pin "1")
+    (instances
+      (project "mqtt-power-control-interface"
+        (path "/23700ef1-6085-46e5-b227-871d4be6e7a6"
+          (reference "#PWR013") (unit 1)
+        )
+        (path "/23700ef1-6085-46e5-b227-871d4be6e7a6/9a6b2a70-b072-4ffe-942c-277ad77cced3"
+          (reference "#PWR03") (unit 1)
+        )
+      )
+    )
+  )
+  (symbol (lib_id "power:GND") (at 55.88 85.09 0) (unit 1)
+    (in_bom yes) (on_board yes) (dnp no) (fields_autoplaced)
+    (property "Reference" "#PWR013" (at 55.88 91.44 0)
+      (effects (font (size 1.27 1.27)) hide)
+    )
+    (property "Value" "GND" (at 55.88 90.17 0)
+      (effects (font (size 1.27 1.27)))
+    )
+    (property "Footprint" "" (at 55.88 85.09 0)
+      (effects (font (size 1.27 1.27)) hide)
+    )
+    (property "Datasheet" "" (at 55.88 85.09 0)
+      (effects (font (size 1.27 1.27)) hide)
+    )
+    (pin "1")
+    (instances
+      (project "mqtt-power-control-interface"
+        (path "/23700ef1-6085-46e5-b227-871d4be6e7a6"
+          (reference "#PWR013") (unit 1)
+        )
+        (path "/23700ef1-6085-46e5-b227-871d4be6e7a6/9a6b2a70-b072-4ffe-942c-277ad77cced3"
+          (reference "#PWR08") (unit 1)
+        )
+      )
+    )
+  )
+  (symbol (lib_id "power:GND") (at 22.86 45.72 0) (unit 1)
+    (in_bom yes) (on_board yes) (dnp no) (fields_autoplaced)
+    (property "Reference" "#PWR013" (at 22.86 52.07 0)
+      (effects (font (size 1.27 1.27)) hide)
+    )
+    (property "Value" "GND" (at 22.86 50.8 0)
+      (effects (font (size 1.27 1.27)))
+    )
+    (property "Footprint" "" (at 22.86 45.72 0)
+      (effects (font (size 1.27 1.27)) hide)
+    )
+    (property "Datasheet" "" (at 22.86 45.72 0)
+      (effects (font (size 1.27 1.27)) hide)
+    )
+    (pin "1")
+    (instances
+      (project "mqtt-power-control-interface"
+        (path "/23700ef1-6085-46e5-b227-871d4be6e7a6"
+          (reference "#PWR013") (unit 1)
+        )
+        (path "/23700ef1-6085-46e5-b227-871d4be6e7a6/9a6b2a70-b072-4ffe-942c-277ad77cced3"
+          (reference "#PWR07") (unit 1)
+        )
+      )
+    )
+  )
   (symbol (lib_id "power:GND") (at 22.86 33.02 0) (unit 1)
     (in_bom yes) (on_board yes) (dnp no) (fields_autoplaced)
@@
         )
       )
+    )
+  )
+  (symbol (lib_id "power:GND") (at 22.86 71.12 0) (unit 1)
+    (in_bom yes) (on_board yes) (dnp no) (fields_autoplaced)
+    (property "Reference" "#PWR013" (at 22.86 77.47 0)
+      (effects (font (size 1.27 1.27)) hide)
+    )
+    (property "Value" "GND" (at 22.86 76.2 0)
+      (effects (font (size 1.27 1.27)))
+    )
+    (property "Footprint" "" (at 22.86 71.12 0)
+      (effects (font (size 1.27 1.27)) hide)
+    )
+    (property "Datasheet" "" (at 22.86 71.12 0)
+      (effects (font (size 1.27 1.27)) hide)
+    )
+    (pin "1")
+    (instances
+      (project "mqtt-power-control-interface"
+        (path "/23700ef1-6085-46e5-b227-871d4be6e7a6"
+          (reference "#PWR013") (unit 1)
+        )
+        (path "/23700ef1-6085-46e5-b227-871d4be6e7a6/9a6b2a70-b072-4ffe-942c-277ad77cced3"
+          (reference "#PWR05") (unit 1)
+        )
+      )
+    )
+  )
+  (symbol (lib_id "power:GND") (at 88.9 71.12 0) (unit 1)
+    (in_bom yes) (on_board yes) (dnp no) (fields_autoplaced)
+    (property "Reference" "#PWR013" (at 88.9 77.47 0)
+      (effects (font (size 1.27 1.27)) hide)
+    )
+    (property "Value" "GND" (at 88.9 76.2 0)
+      (effects (font (size 1.27 1.27)))
+    )
+    (property "Footprint" "" (at 88.9 71.12 0)
+      (effects (font (size 1.27 1.27)) hide)
+    )
+    (property "Datasheet" "" (at 88.9 71.12 0)
+      (effects (font (size 1.27 1.27)) hide)
+    )
+    (pin "1")
+    (instances
+      (project "mqtt-power-control-interface"
+        (path "/23700ef1-6085-46e5-b227-871d4be6e7a6"
+          (reference "#PWR013") (unit 1)
+        )
+        (path "/23700ef1-6085-46e5-b227-871d4be6e7a6/9a6b2a70-b072-4ffe-942c-277ad77cced3"
+          (reference "#PWR04") (unit 1)
+        )
+      )
